File: Proyectos/Steppers/CAD/Stepper_2_0/Stepper_2_0.sch (EAGLE design)
At the start: 79 parts

Commit message: Steppers:
Corrección de esquemático
Parts:
- removed U$1: DUE(NOSPI), JoshParts:DUE(NOSPI)
- added C10: 0.1u, SparkFun-Passives:CAP1206
- added C7: 10u, rcl:CPOL-EUE2-4
- added C8: 10u, SparkFun-Passives:CAP1206
- added C9: 4.7u, SparkFun-Passives:CAP1206
- added DUE1: DUE(NOSPI), JoshParts:DUE(NOSPI)
- added JP19: (no value), pinhead:PINHD-1X2
- added L1: (no value), WE-CBF:WE-CBF-742792118_1206
- added LED13, LED14: RED, adafruit:LEDSMT1206
- added PS1: VX78-500, Steppers:VX78-500
- added R13, R14: 150, SparkFun-Resistors:RESISTOR1206
- added TB7: TB_HEAD_3.5MM_01X02, Steppers:TB_HEAD_3.5MM_01X02
- JP11, JP12, JP2, JP3: device pinhead:PINHD-1X2 -> pinhead:PINHD-2X3
- JP13, JP16, JP4, JP6: device pinhead:PINHD-2X3 -> pinhead:PINHD-1X2
- LED10, LED2: value RED -> GREEN
- LED5: value GREEN -> RED
- R7, R8: value 150 -> 1K
Connections:
- removed net N$25 (its old number): LED5.A
- removed net N$36 (its old number): LED7.A
- removed net N$64 (its old number): JP6.6, PL6.MS3
- removed net N$65 (its old number): JP6.4, PL6.MS2
- removed net N$66 (its old number): JP6.2, PL6.MS1
- new net 9V: C10.2, C8.2, C9.2, JP19.1, L1.2, LED7.A
- new net N$14: LED2.A
- new net N$34: LED12.C, R9.1
- new net N$35: LED9.C, R12.1
- new net N$47: LED10.A
- new net N$6: JP2.6, PL2.MS3
- new net N$67: L1.1, PS1.P$2
- new net N$7: JP2.4, PL2.MS2
- new net N$8: JP2.2, PL2.MS1
- new net VIN: DUE1.VIN, JP19.2, LED8.A
- net 3V3: now also DUE1.3V3, JP11.1, JP11.3, JP11.5, JP12.1, JP12.3, JP12.5, JP2.1, JP2.3, JP2.5, JP3.1, JP3.3, JP3.5; no longer JP13.1, JP13.3, JP13.5, JP16.1, JP16.3, JP16.5, JP4.1, JP4.3, JP4.5, JP6.1, JP6.3, JP6.5, U$1.3V3
- net GND: now also C10.1, C7.-, C8.1, C9.1, DUE1.GND_1, DUE1.GND_2, DUE1.GND_A, DUE1.GND_B, JP13.2, JP16.2, JP4.2, JP6.2, PS1.P$3, R1.2, R11.2, R3.2, R7.2, R9.2, TB7.P$2; no longer JP11.2, JP12.2, JP2.2, JP3.2, R12.2, R4.2, R6.2, U$1.GND_1, U$1.GND_2, U$1.GND_A, U$1.GND_B
- net M1_DIR: now also PL1.DIR; no longer PL6.DIR
- net M1_EN: now also PL1.!EN; no longer PL6.!EN
- net M1_LED: now also LED4.A, R4.2; no longer LED2.A, R1.2
- net M1_SL: now also JP4.1; no longer JP7.1
- net M1_SR: now also JP5.1; no longer JP8.1
- net M1_STEP: now also PL1.STP; no longer PL6.STP
- net M2_DIR: now also PL2.DIR; no longer PL1.DIR
- net M2_EN: now also PL2.!EN; no longer PL1.!EN
- net M2_LED: now also LED5.A, R5.2; no longer LED4.A, R3.2
- net M2_SL: now also JP6.1; no longer JP2.1
- net M2_SR: now also JP7.1; no longer JP3.1
- net M2_STEP: now also PL2.STP; no longer PL1.STP
- net M3_DIR: now also PL3.DIR; no longer PL2.DIR
- net M3_EN: now also PL3.!EN; no longer PL2.!EN
- net M3_LED: now also R6.2; no longer R5.2
- net M3_SL: now also JP8.1; no longer JP5.1
- net M3_STEP: now also PL3.STP; no longer PL2.STP
- net M4_DIR: now also PL4.DIR; no longer PL3.DIR
- net M4_EN: now also PL4.!EN; no longer PL3.!EN
- net M4_LED: now also LED12.A, R12.2; no longer LED8.A, R7.2
- net M4_SL: now also JP13.1; no longer JP11.1
- net M4_SR: now also JP14.1; no longer JP12.1
- net M4_STEP: now also PL4.STP; no longer PL3.STP
- net M5_DIR: now also PL5.DIR; no longer PL4.DIR
- net M5_EN: now also PL5.!EN; no longer PL4.!EN
- net M5_LED: now also LED13.A, R13.2; no longer LED10.A, R9.2
- net M5_SL: now also JP15.1; no longer JP14.1
- net M5_SR: now also JP16.1; no longer JP15.1
- net M5_STEP: now also PL5.STP; no longer PL4.STP
- net M6_DIR: now also PL6.DIR; no longer PL5.DIR
- net M6_EN: now also PL6.!EN; no longer PL5.!EN
- net M6_LED: now also LED14.A, R14.2; no longer LED12.A, R11.2
- net M6_STEP: now also PL6.STP; no longer PL5.STP
- net N$10: now also LED5.C, R2.1; no longer LED4.C, R4.1
- net N$11: now also R4.1; no longer R1.1
- net N$13: now also LED2.C, R5.1; no longer LED3.C, R3.1
- net N$20: now also JP3.6, PL3.MS3; no longer JP4.6, PL2.MS3
- net N$21: now also JP3.4, PL3.MS2; no longer JP4.4, PL2.MS2
- net N$22: now also JP3.2, PL3.MS1; no longer JP4.2, PL2.MS1
- net N$23: now also R3.1; no longer R6.1
- net N$24: now also LED3.C, R6.1; no longer LED5.C, R5.1
- net N$31: now also PL4.MS3; no longer PL3.MS3
- net N$32: now also PL4.MS2; no longer PL3.MS2
- net N$33: now also PL4.MS1; no longer PL3.MS1
- net N$42: now also JP11.6, PL5.MS3; no longer JP13.6, PL4.MS3
- net N$43: now also JP11.4, PL5.MS2; no longer JP13.4, PL4.MS2
- net N$44: now also JP11.2, PL5.MS1; no longer JP13.2, PL4.MS1
- net N$45: now also LED13.C; no longer LED10.C
- net N$46: now also LED10.C, R13.1; no longer LED9.C, R9.1
- net N$53: now also JP12.6, PL6.MS3; no longer JP16.6, PL5.MS3
- net N$54: now also JP12.4, PL6.MS2; no longer JP16.4, PL5.MS2
- net N$55: now also JP12.2, PL6.MS1; no longer JP16.2, PL5.MS1
- net N$56: now also LED14.C, R11.1; no longer LED12.C, R12.1
- net N$61: now also R14.1; no longer R11.1
- net N$9: now also LED4.C, R1.1; no longer LED2.C, R2.1
- net VCC: now also C7.+, PS1.P$1, TB7.P$3
Other:
- note removed: "1"
- note removed: "2"
- note removed: "3"
- note removed: "4"
- note removed: "5"
- note removed: "6"
- note removed: "Control Manual"
- note removed: "Indicador de uso"
- note removed: "Sensores Final de carrera"
- moved on the sheet: C1, C2, C3, C4, C5, C6, JP1, JP10, JP14, JP15, JP17, JP18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

Commit message: Steppers:
Avance en PCB final, asignación de pines DUE.
Parts:
- added H1, H2, H3, H4, H5, H6: STAND-OFF, SparkFun-Electromechanical:STAND-OFF
Connections:
- removed net N$12: LED1.A
- removed net N$14: LED2.A
- removed net N$25: LED3.A
- removed net N$36: LED9.A
- removed net N$47: LED10.A
- removed net N$63: LED11.A
- new net N$97: DUE1.23
- new net N$98: DUE1.22
- net 3V3: now also LED1.A, LED10.A, LED11.A, LED2.A, LED3.A, LED9.A
- net M1_DIR: now also DUE1.52
- net M1_EN: now also DUE1.51
- net M1_SL: now also DUE1.34
- net M1_SR: now also DUE1.35
- net M1_STEP: now also DUE1.53
- net M2_DIR: now also DUE1.50
- net M2_EN: now also DUE1.49
- net M2_SL: now also DUE1.32
- net M2_SR: now also DUE1.33
- net M2_STEP: now also DUE1.48
- net M3_DIR: now also DUE1.46
- net M3_EN: now also DUE1.45
- net M3_SL: now also DUE1.30
- net M3_SR: now also DUE1.31
- net M3_STEP: now also DUE1.47
- net M4_DIR: now also DUE1.44
- net M4_EN: now also DUE1.43
- net M4_SL: now also DUE1.28
- net M4_SR: now also DUE1.29
- net M4_STEP: now also DUE1.42
- net M5_DIR: now also DUE1.40
- net M5_EN: now also DUE1.39
- net M5_SL: now also DUE1.26
- net M5_SR: now also DUE1.27
- net M5_STEP: now also DUE1.41
- net M6_DIR: now also DUE1.38
- net M6_EN: now also DUE1.37
- net M6_SL: now also DUE1.24
- net M6_SR: now also DUE1.25
- net M6_STEP: now also DUE1.36
- net N$20: now also JP3.2; no longer JP3.6
- net N$22: now also JP3.6; no longer JP3.2
- net N$31: now also JP10.2; no longer JP10.6
- net N$33: now also JP10.6; no longer JP10.2
- net N$42: now also JP11.2; no longer JP11.6
- net N$44: now also JP11.6; no longer JP11.2
- net N$53: now also PL6.MS1; no longer PL6.MS3
- net N$55: now also PL6.MS3; no longer PL6.MS1
- net N$6: now also JP2.2; no longer JP2.6
- net N$64: now also JP1.2; no longer JP1.6
- net N$66: now also JP1.6; no longer JP1.2
- net N$8: now also JP2.6; no longer JP2.2

Commit message: Steppers:
Se finaliza el esquemático y PCB de forma funcional.
Parts:
- removed H6: STAND-OFF, SparkFun-Electromechanical:STAND-OFF
Connections:
- removed net N$97: DUE1.23
- removed net N$98: DUE1.22
- net M1_BTNL: now also DUE1.2
- net M1_BTNR: now also DUE1.3
- net M1_LED: now also DUE1.13
- net M1_MVEL: now also DUE1.A0
- net M2_BTNL: now also DUE1.4
- net M2_BTNR: now also DUE1.5
- net M2_LED: now also DUE1.12
- net M2_MVEL: now also DUE1.A1
- net M3_BTNL: now also DUE1.6
- net M3_BTNR: now also DUE1.7
- net M3_LED: now also DUE1.11
- net M3_MVEL: now also DUE1.A2
- net M4_BTNL: now also DUE1.RX1
- net M4_BTNR: now also DUE1.TX1
- net M4_LED: now also DUE1.10
- net M4_MVEL: now also DUE1.A3
- net M5_BTNL: now also DUE1.RX2
- net M5_BTNR: now also DUE1.TX2
- net M5_LED: now also DUE1.9
- net M5_MVEL: now also DUE1.A4
- net M6_BTNL: now also DUE1.RX3
- net M6_BTNR: now also DUE1.TX3
- net M6_LED: now also DUE1.8
- net M6_MVEL: now also DUE1.A5
Changed lines of the file:
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@@
 <setting verticaltext="up"/>
 </settings>
-<grid distance="0.1" unitdist="inch" unit="inch" style="lines" multiple="1" display="yes" altdistance="0.01" altunitdist="inch" altunit="inch"/>
+<grid distance="0.1" unitdist="inch" unit="inch" style="lines" multiple="1" display="no" altdistance="0.01" altunitdist="inch" altunit="inch"/>
 <layers>
 <layer number="1" name="Top" color="4" fill="1" visible="no" active="no"/>
@@
 <part name="H4" library="SparkFun-Electromechanical" deviceset="STAND-OFF" device=""/>
 <part name="H5" library="SparkFun-Electromechanical" deviceset="STAND-OFF" device=""/>
-<part name="H6" library="SparkFun-Electromechanical" deviceset="STAND-OFF" device=""/>
 </parts>
 <sheets>
@@
 <instance part="H4" gate="G$1" x="256.54" y="190.5"/>
 <instance part="H5" gate="G$1" x="256.54" y="200.66"/>
-<instance part="H6" gate="G$1" x="256.54" y="195.58"/>
 </instances>
 <busses>
@@
 <label x="116.84" y="127" size="1.778" layer="95"/>
 </segment>
+<segment>
+<pinref part="DUE1" gate="G$1" pin="3"/>
+<wire x1="53.34" y1="269.24" x2="53.34" y2="279.4" width="0.1524" layer="91"/>
+<label x="53.34" y="269.24" size="1.778" layer="95" rot="R90"/>
+</segment>
 </net>
 <net name="M1_BTNL" class="0">
@@
 <label x="116.84" y="137.16" size="1.778" layer="95"/>
 </segment>
+<segment>
+<pinref part="DUE1" gate="G$1" pin="2"/>
+<wire x1="50.8" y1="269.24" x2="50.8" y2="279.4" width="0.1524" layer="91"/>
+<label x="50.8" y="269.24" size="1.778" layer="95" rot="R90"/>
+</segment>
 </net>
 <net name="M1_MVEL" class="0">
@@
 <wire x1="137.16" y1="149.86" x2="116.84" y2="149.86" width="0.1524" layer="91"/>
 <label x="116.84" y="149.86" size="1.778" layer="95"/>
+</segment>
+<segment>
+<pinref part="DUE1" gate="G$1" pin="A0"/>
+<wire x1="35.56" y1="180.34" x2="35.56" y2="170.18" width="0.1524" layer="91"/>
+<label x="35.56" y="170.18" size="1.778" layer="95" rot="R90"/>
 </segment>
 </net>
@@
 <label x="154.94" y="137.16" size="1.778" layer="95"/>
 </segment>
+<segment>
+<pinref part="DUE1" gate="G$1" pin="13"/>
+<wire x1="78.74" y1="269.24" x2="78.74" y2="279.4" width="0.1524" layer="91"/>
+<label x="78.74" y="269.24" size="1.778" layer="95" rot="R90"/>
+</segment>
 </net>
 <net name="N$11" class="0">
@@
 <wire x1="137.16" y1="93.98" x2="116.84" y2="93.98" width="0.1524" layer="91"/>
 <label x="116.84" y="93.98" size="1.778" layer="95"/>
+</segment>
+<segment>
+<pinref part="DUE1" gate="G$1" pin="A1"/>
+<wire x1="38.1" y1="180.34" x2="38.1" y2="170.18" width="0.1524" layer="91"/>
+<label x="38.1" y="170.18" size="1.778" layer="95" rot="R90"/>
 </segment>
 </net>
@@
 <label x="116.84" y="81.28" size="1.778" layer="95"/>
 </segment>
+<segment>
+<pinref part="DUE1" gate="G$1" pin="4"/>
+<wire x1="55.88" y1="269.24" x2="55.88" y2="279.4" width="0.1524" layer="91"/>
+<label x="55.88" y="269.24" size="1.778" layer="95" rot="R90"/>
+</segment>
 </net>
 <net name="M2_BTNR" class="0">
@@
 <junction x="129.54" y="71.12"/>
 <label x="116.84" y="71.12" size="1.778" layer="95"/>
+</segment>
+<segment>
+<pinref part="DUE1" gate="G$1" pin="5"/>
+<wire x1="58.42" y1="269.24" x2="58.42" y2="279.4" width="0.1524" layer="91"/>
+<label x="58.42" y="269.24" size="1.778" layer="95" rot="R90"/>
 </segment>
 </net>
@@
 <label x="154.94" y="81.28" size="1.778" layer="95"/>
 </segment>
+<segment>
+<pinref part="DUE1" gate="G$1" pin="12"/>
+<wire x1="76.2" y1="269.24" x2="76.2" y2="279.4" width="0.1524" layer="91"/>
+<label x="76.2" y="269.24" size="1.778" layer="95" rot="R90"/>
+</segment>
 </net>
 <net name="M3_EN" class="0">
@@
 <label x="154.94" y="25.4" size="1.778" layer="95"/>
 </segment>
+<segment>
+<pinref part="DUE1" gate="G$1" pin="11"/>
+<wire x1="73.66" y1="269.24" x2="73.66" y2="279.4" width="0.1524" layer="91"/>
+<label x="73.66" y="269.24" size="1.778" layer="95" rot="R90"/>
+</segment>
 </net>
 <net name="M3_MVEL" class="0">
@@
 <wire x1="137.16" y1="38.1" x2="116.84" y2="38.1" width="0.1524" layer="91"/>
 <label x="116.84" y="38.1" size="1.778" layer="95"/>
+</segment>
+<segment>
+<pinref part="DUE1" gate="G$1" pin="A2"/>
+<wire x1="40.64" y1="180.34" x2="40.64" y2="170.18" width="0.1524" layer="91"/>
+<label x="40.64" y="170.18" size="1.778" layer="95" rot="R90"/>
 </segment>
 </net>
@@
 <label x="116.84" y="25.4" size="1.778" layer="95"/>
 </segment>
+<segment>
+<pinref part="DUE1" gate="G$1" pin="6"/>
+<wire x1="60.96" y1="269.24" x2="60.96" y2="279.4" width="0.1524" layer="91"/>
+<label x="60.96" y="269.24" size="1.778" layer="95" rot="R90"/>
+</segment>
 </net>
 <net name="M3_BTNR" class="0">
@@
 <label x="116.84" y="15.24" size="1.778" layer="95"/>
 </segment>
+<segment>
+<pinref part="DUE1" gate="G$1" pin="7"/>
+<wire x1="63.5" y1="269.24" x2="63.5" y2="279.4" width="0.1524" layer="91"/>
+<label x="63.5" y="269.24" size="1.778" layer="95" rot="R90"/>
+</segment>
 </net>
 <net name="M6_EN" class="0">
@@
 <wire x1="317.5" y1="38.1" x2="297.18" y2="38.1" width="0.1524" layer="91"/>
 <label x="297.18" y="38.1" size="1.778" layer="95"/>
+</segment>
+<segment>
+<pinref part="DUE1" gate="G$1" pin="A5"/>
+<wire x1="48.26" y1="180.34" x2="48.26" y2="170.18" width="0.1524" layer="91"/>
+<label x="48.26" y="170.18" size="1.778" layer="95" rot="R90"/>
 </segment>
 </net>
@@
 <label x="297.18" y="25.4" size="1.778" layer="95"/>
 </segment>
+<segment>
+<pinref part="DUE1" gate="G$1" pin="RX3"/>
+<wire x1="17.78" y1="236.22" x2="7.62" y2="236.22" width="0.1524" layer="91"/>
+<label x="7.62" y="236.22" size="1.778" layer="95"/>
+</segment>
 </net>
 <net name="M6_BTNR" class="0">
@@
 <junction x="309.88" y="15.24"/>
 <label x="297.18" y="15.24" size="1.778" layer="95"/>
+</segment>
+<segment>
+<pinref part="DUE1" gate="G$1" pin="TX3"/>
+<wire x1="17.78" y1="238.76" x2="7.62" y2="238.76" width="0.1524" layer="91"/>
+<label x="7.62" y="238.76" size="1.778" layer="95"/>
 </segment>
 </net>
@@
 <label x="335.28" y="25.4" size="1.778" layer="95"/>
 </segment>
+<segment>
+<pinref part="DUE1" gate="G$1" pin="8"/>
+<wire x1="66.04" y1="269.24" x2="66.04" y2="279.4" width="0.1524" layer="91"/>
+<label x="66.04" y="269.24" size="1.778" layer="95" rot="R90"/>
+</segment>
 </net>
 <net name="M5_EN" class="0">
@@
 <wire x1="317.5" y1="93.98" x2="297.18" y2="93.98" width="0.1524" layer="91"/>
 <label x="297.18" y="93.98" size="1.778" layer="95"/>
+</segment>
+<segment>
+<pinref part="DUE1" gate="G$1" pin="A4"/>
+<wire x1="45.72" y1="180.34" x2="45.72" y2="170.18" width="0.1524" layer="91"/>
+<label x="45.72" y="170.18" size="1.778" layer="95" rot="R90"/>
 </segment>
 </net>
@@
 <label x="297.18" y="81.28" size="1.778" layer="95"/>
 </segment>
+<segment>
+<pinref part="DUE1" gate="G$1" pin="RX2"/>
+<wire x1="17.78" y1="231.14" x2="7.62" y2="231.14" width="0.1524" layer="91"/>
+<label x="7.62" y="231.14" size="1.778" layer="95"/>
+</segment>
 </net>
 <net name="M5_BTNR" class="0">
@@
 <junction x="309.88" y="71.12"/>
 <label x="297.18" y="71.12" size="1.778" layer="95"/>
+</segment>
+<segment>
+<pinref part="DUE1" gate="G$1" pin="TX2"/>
+<wire x1="17.78" y1="233.68" x2="7.62" y2="233.68" width="0.1524" layer="91"/>
+<label x="7.62" y="233.68" size="1.778" layer="95"/>
 </segment>
 </net>
@@
 <label x="335.28" y="81.28" size="1.778" layer="95"/>
 </segment>
+<segment>
+<pinref part="DUE1" gate="G$1" pin="9"/>
+<wire x1="68.58" y1="269.24" x2="68.58" y2="279.4" width="0.1524" layer="91"/>
+<label x="68.58" y="269.24" size="1.778" layer="95" rot="R90"/>
+</segment>
 </net>
 <net name="M4_LED" class="0">
@@
 <label x="335.28" y="137.16" size="1.778" layer="95"/>
 </segment>
+<segment>
+<pinref part="DUE1" gate="G$1" pin="10"/>
+<wire x1="71.12" y1="269.24" x2="71.12" y2="279.4" width="0.1524" layer="91"/>
+<label x="71.12" y="269.24" size="1.778" layer="95" rot="R90"/>
+</segment>
 </net>
 <net name="M4_MVEL" class="0">
@@
 <wire x1="317.5" y1="149.86" x2="297.18" y2="149.86" width="0.1524" layer="91"/>
 <label x="297.18" y="149.86" size="1.778" layer="95"/>
+</segment>
+<segment>
+<pinref part="DUE1" gate="G$1" pin="A3"/>
+<wire x1="43.18" y1="180.34" x2="43.18" y2="170.18" width="0.1524" layer="91"/>
+<label x="43.18" y="170.18" size="1.778" layer="95" rot="R90"/>
 </segment>
 </net>
@@
 <label x="297.18" y="137.16" size="1.778" layer="95"/>
 </segment>
+<segment>
+<pinref part="DUE1" gate="G$1" pin="RX1"/>
+<wire x1="17.78" y1="226.06" x2="7.62" y2="226.06" width="0.1524" layer="91"/>
+<label x="7.62" y="226.06" size="1.778" layer="95"/>
+</segment>
 </net>
 <net name="M4_BTNR" class="0">
@@
 <junction x="309.88" y="127"/>
 <label x="297.18" y="127" size="1.778" layer="95"/>
+</segment>
+<segment>
+<pinref part="DUE1" gate="G$1" pin="TX1"/>
+<wire x1="17.78" y1="228.6" x2="7.62" y2="228.6" width="0.1524" layer="91"/>
+<label x="7.62" y="228.6" size="1.778" layer="95"/>
 </segment>
 </net>
@@
 </segment>
 </net>
-<net name="N$97" class="0">
-<segment>
-<pinref part="DUE1" gate="G$1" pin="23"/>
-<wire x1="99.06" y1="261.62" x2="88.9" y2="261.62" width="0.1524" layer="91"/>
-<label x="88.9" y="261.62" size="1.778" layer="95"/>
-</segment>
-</net>
-<net name="N$98" class="0">
-<segment>
-<pinref part="DUE1" gate="G$1" pin="22"/>
-<wire x1="99.06" y1="264.16" x2="88.9" y2="264.16" width="0.1524" layer="91"/>
-<label x="88.9" y="264.16" size="1.778" layer="95"/>
-</segment>
-</net>

Commit message: Steppers:
Se añaden pads para testeo de voltajes y conexión de 5V para ventilador.
Parts:
- added JP20: (no value), pinhead:PINHD-1X2
Connections:
- new net 5V: DUE1.5V, JP20.2
- net GND: now also JP20.1
